Commit message: urdf update && reward func minor fix && obs man viz fix

File: source/isaaclab_assets/data/Robots/Tocabi/urdf/dyros_tocabi.urdf (robot description, URDF)
Before this commit: robot tocabi, 36 links, 35 joints
Links:
- link L_AnkleCenter_Link: mass 2.833 -> 2.51
- link L_AnkleRoll_Link: mass 2.1 -> 1.26426
- link L_Foot_Link: mass 2.350 -> 2.326
- link L_Knee_Link: mass 2.614 -> 3.883
- link L_Thigh_Link: mass 5.65 -> 5.366
- link Pelvis_Link: mass 12.9 -> 12.19525
- link R_AnkleCenter_Link: mass 2.833 -> 2.51
- link R_AnkleRoll_Link: mass 2.1 -> 1.26426
- link R_Foot_Link: mass 2.35 -> 2.326
- link R_Knee_Link: mass 2.614 -> 3.883
- link R_Thigh_Link: mass 5.65 -> 5.366
- link Waist1_Link: mass 6.477 -> 0.89722
- link Waist2_Link: mass 3.881 -> 3.752
Joints:
- joint L_AnklePitch_Joint: limit lower=-0.8 upper=0.5 effort=222 velocity=20 -> lower=-3.14 upper=3.14 effort=222 velocity=20
- joint L_AnkleRoll_Joint: limit lower=-0.6 upper=0.6 effort=166 velocity=20 -> lower=-3.14 upper=3.14 effort=166 velocity=20
- joint L_HipPitch_Joint: limit lower=-1.0 upper=0.5 effort=263 velocity=20 -> lower=-3.14 upper=3.14 effort=263 velocity=20
- joint L_HipRoll_Joint: limit lower=-0.5 upper=0.5 effort=232 velocity=20 -> lower=-3.14 upper=3.14 effort=232 velocity=20
- joint L_HipYaw_Joint: limit lower=-0.3 upper=0.3 effort=333 velocity=20.0 -> lower=-3.14 upper=3.14 effort=333 velocity=20.0
- joint L_Knee_Joint: limit lower=-0.3 upper=1.2 effort=289 velocity=20 -> lower=-3.14 upper=3.14 effort=289 velocity=20
- joint R_AnklePitch_Joint: limit lower=-0.8 upper=0.5 effort=222 velocity=20 -> lower=-3.14 upper=3.14 effort=222 velocity=20
- joint R_AnkleRoll_Joint: limit lower=-0.6 upper=0.6 effort=166 velocity=20 -> lower=-3.14 upper=3.14 effort=166 velocity=20
- joint R_HipPitch_Joint: limit lower=-1.0 upper=0.5 effort=263 velocity=20 -> lower=-3.14 upper=3.14 effort=263 velocity=20
- joint R_HipRoll_Joint: limit lower=-0.5 upper=0.5 effort=232 velocity=20 -> lower=-3.14 upper=3.14 effort=232 velocity=20
- joint R_HipYaw_Joint: limit lower=-0.3 upper=0.3 effort=333 velocity=20 -> lower=-3.14 upper=3.14 effort=333 velocity=20
- joint R_Knee_Joint: limit lower=-0.3 upper=1.2 effort=289 velocity=20 -> lower=-3.14 upper=3.14 effort=289 velocity=20
